File: 12v_detect.kicad_sch (KiCad schematic)
At the start: 3 parts, among them Q6 BS170

Commit message: Most of the layout completed
Parts:
- renumbered Q6 to Q4, R14 to R13, R17 to R14
Changed lines of the file:
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@@
 		(dnp no)
 		(fields_autoplaced yes)
-		(property "Reference" "#PWR52"
+		(property "Reference" "#PWR043"
 			(at 133.35 102.87 0)
 			(effects
@@
 			(project ""
 				(path "/40f6f48c-88df-4c09-997b-20b4a32eb379/cff5f72d-d49c-4426-884a-a2476ea7661a"
-					(reference "#PWR52")
+					(reference "#PWR043")
 					(unit 1)
 				)
@@
 		(dnp no)
 		(fields_autoplaced yes)
-		(property "Reference" "Q6"
+		(property "Reference" "Q4"
 			(at 137.16 83.8199 0)
 			(effects
@@
 			(project ""
 				(path "/40f6f48c-88df-4c09-997b-20b4a32eb379/cff5f72d-d49c-4426-884a-a2476ea7661a"
-					(reference "Q6")
+					(reference "Q4")
 					(unit 1)
 				)
@@
 		(dnp no)
 		(fields_autoplaced yes)
-		(property "Reference" "R17"
+		(property "Reference" "R14"
 			(at 124.46 87.6299 0)
 			(effects
@@
 			(project ""
 				(path "/40f6f48c-88df-4c09-997b-20b4a32eb379/cff5f72d-d49c-4426-884a-a2476ea7661a"
-					(reference "R17")
+					(reference "R14")
 					(unit 1)
 				)
@@
 		(dnp no)
 		(fields_autoplaced yes)
-		(property "Reference" "R14"
+		(property "Reference" "R13"
 			(at 135.89 69.8499 0)
 			(effects
@@
 			(project ""
 				(path "/40f6f48c-88df-4c09-997b-20b4a32eb379/cff5f72d-d49c-4426-884a-a2476ea7661a"
-					(reference "R14")
-					(unit 1)
-				)
+					(reference "R13")
+					(unit 1)
+				)
