File: 12v_switched_relay.kicad_sch (KiCad schematic)
At the start: 4 parts, among them K3 SRD-12VDC-SL-C, Q3 BS170

Commit message: Various fixes
Signed-off-by: Tobias de Bruijn <t.debruijn@array21.dev>
Parts:
- K4: renamed from K3; footprint SRD-12VDC-SL-C:RELAY_SRD-12VDC-SL-C -> footprints:RELAY_SRD-12VDC-SL-C
- R8: renamed from R7; value R -> 10K; footprint (none) -> Resistor_SMD:R_1206_3216Metric
- renumbered D5 to D6, Q3 to Q4
Changed lines of the file:
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@@
 (kicad_sch
-	(version 20231120)
+	(version 20250114)
 	(generator "eeschema")
-	(generator_version "8.0")
+	(generator_version "9.0")
 	(paper "A4")
 	(junction
@@
 		(dnp no)
 		(fields_autoplaced yes)
-		(property "Reference" "#PWR3"
+		(property "Reference" "#PWR28"
 			(at 133.35 93.98 0)
 			(effects
@@
 		(instances
 			(project "twingo_aa"
-				(path "/40f6f48c-88df-4c09-997b-20b4a32eb379/07c20ec4-560b-4446-9e27-966b386d70c5"
-					(reference "#PWR3")
-					(unit 1)
-				)
 				(path "/40f6f48c-88df-4c09-997b-20b4a32eb379/b9f9eead-f3cf-4016-8c85-192ff17ff478"
 					(reference "#PWR28")
@@
 		(dnp no)
 		(fields_autoplaced yes)
-		(property "Reference" "D5"
+		(property "Reference" "D6"
 			(at 135.89 95.2499 90)
 			(effects
@@
 		(instances
 			(project "twingo_aa"
-				(path "/40f6f48c-88df-4c09-997b-20b4a32eb379/07c20ec4-560b-4446-9e27-966b386d70c5"
-					(reference "D5")
-					(unit 1)
-				)
 				(path "/40f6f48c-88df-4c09-997b-20b4a32eb379/b9f9eead-f3cf-4016-8c85-192ff17ff478"
 					(reference "D6")
@@
 		(dnp no)
 		(fields_autoplaced yes)
-		(property "Reference" "Q3"
+		(property "Reference" "Q4"
 			(at 137.16 111.7599 0)
 			(effects
@@
 		(instances
 			(project "twingo_aa"
-				(path "/40f6f48c-88df-4c09-997b-20b4a32eb379/07c20ec4-560b-4446-9e27-966b386d70c5"
-					(reference "Q3")
-					(unit 1)
-				)
 				(path "/40f6f48c-88df-4c09-997b-20b4a32eb379/b9f9eead-f3cf-4016-8c85-192ff17ff478"
 					(reference "Q4")
@@
 		(dnp no)
 		(fields_autoplaced yes)
-		(property "Reference" "#PWR30"
+		(property "Reference" "#PWR32"
 			(at 133.35 127 0)
 			(effects
@@
 		(instances
 			(project "twingo_aa"
-				(path "/40f6f48c-88df-4c09-997b-20b4a32eb379/07c20ec4-560b-4446-9e27-966b386d70c5"
-					(reference "#PWR30")
-					(unit 1)
-				)
 				(path "/40f6f48c-88df-4c09-997b-20b4a32eb379/b9f9eead-f3cf-4016-8c85-192ff17ff478"
 					(reference "#PWR32")
@@
 		(dnp no)
 		(fields_autoplaced yes)
-		(property "Reference" "R7"
+		(property "Reference" "R8"
 			(at 123.19 115.5699 0)
 			(effects
@@
 			)
 		)
-		(property "Value" "R"
+		(property "Value" "10K"
 			(at 123.19 118.1099 0)
 			(effects
@@
 			)
 		)
-		(property "Footprint" ""
+		(property "Footprint" "Resistor_SMD:R_1206_3216Metric"
 			(at 118.872 116.84 90)
 			(effects
@@
 		(instances
 			(project "twingo_aa"
-				(path "/40f6f48c-88df-4c09-997b-20b4a32eb379/07c20ec4-560b-4446-9e27-966b386d70c5"
-					(reference "R7")
-					(unit 1)
-				)
 				(path "/40f6f48c-88df-4c09-997b-20b4a32eb379/b9f9eead-f3cf-4016-8c85-192ff17ff478"
 					(reference "R8")
@@
 		(dnp no)
 		(fields_autoplaced yes)
-		(property "Reference" "K3"
+		(property "Reference" "K4"
 			(at 153.67 82.55 0)
 			(effects
@@
 			)
 		)
-		(property "Footprint" "SRD-12VDC-SL-C:RELAY_SRD-12VDC-SL-C"
+		(property "Footprint" "footprints:RELAY_SRD-12VDC-SL-C"
 			(at 153.67 95.25 0)
 			(effects
@@
 		(instances
 			(project "twingo_aa"
-				(path "/40f6f48c-88df-4c09-997b-20b4a32eb379/07c20ec4-560b-4446-9e27-966b386d70c5"
-					(reference "K3")
-					(unit 1)
-				)
 				(path "/40f6f48c-88df-4c09-997b-20b4a32eb379/b9f9eead-f3cf-4016-8c85-192ff17ff478"
 					(reference "K4")

Commit message: Most of the layout completed
Parts:
- renumbered K4 to K3, Q4 to Q3
Changed lines of the file:
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@@
 		(dnp no)
 		(fields_autoplaced yes)
-		(property "Reference" "#PWR28"
+		(property "Reference" "#PWR032"
 			(at 133.35 93.98 0)
 			(effects
@@
 			(project "twingo_aa"
 				(path "/40f6f48c-88df-4c09-997b-20b4a32eb379/b9f9eead-f3cf-4016-8c85-192ff17ff478"
-					(reference "#PWR28")
+					(reference "#PWR032")
 					(unit 1)
 				)
@@
 		(dnp no)
 		(fields_autoplaced yes)
-		(property "Reference" "Q4"
+		(property "Reference" "Q3"
 			(at 137.16 111.7599 0)
 			(effects
@@
 			(project "twingo_aa"
 				(path "/40f6f48c-88df-4c09-997b-20b4a32eb379/b9f9eead-f3cf-4016-8c85-192ff17ff478"
-					(reference "Q4")
+					(reference "Q3")
 					(unit 1)
 				)
@@
 		(dnp no)
 		(fields_autoplaced yes)
-		(property "Reference" "#PWR32"
+		(property "Reference" "#PWR033"
 			(at 133.35 127 0)
 			(effects
@@
 			(project "twingo_aa"
 				(path "/40f6f48c-88df-4c09-997b-20b4a32eb379/b9f9eead-f3cf-4016-8c85-192ff17ff478"
-					(reference "#PWR32")
+					(reference "#PWR033")
 					(unit 1)
 				)
@@
 		(dnp no)
 		(fields_autoplaced yes)
-		(property "Reference" "K4"
+		(property "Reference" "K3"
 			(at 153.67 82.55 0)
 			(effects
@@
 			(project "twingo_aa"
 				(path "/40f6f48c-88df-4c09-997b-20b4a32eb379/b9f9eead-f3cf-4016-8c85-192ff17ff478"
-					(reference "K4")
+					(reference "K3")
 					(unit 1)
 				)
