File: 12v_switched_relay_no_pulldown.kicad_sch (KiCad schematic)
At the start: 4 parts, among them K1 SRD-05VDC-SL-C, Q1 BS170

Commit message: Various fixes
Signed-off-by: Tobias de Bruijn <t.debruijn@array21.dev>
Parts:
- removed D3: 1N4007, Diode_THT:D_DO-41_SOD81_P10.16mm_Horizontal, symbol Diode:1N4007
- removed K1: SRD-05VDC-SL-C, footprints:SRD-05VDC-SL-C, symbol SRD-05VDC-SL-C:SRD-05VDC-SL-C
- removed Q1: BS170, Package_TO_SOT_THT:TO-92_Inline, symbol Transistor_FET:BS170
- removed R6: 10K, Resistor_SMD:R_1206_3216Metric, symbol Device:R
- added D5: 1N4007, Diode_THT:D_DO-41_SOD81_P10.16mm_Horizontal, symbol Diode:1N4007
- added K3: SRD-12VDC-SL-C, footprints:RELAY_SRD-12VDC-SL-C, symbol SRD-12VDC-SL-C:SRD-12VDC-SL-C
- added Q3: BS170, Package_TO_SOT_THT:TO-92_Inline, symbol Transistor_FET:BS170
Connections:
- net Com: now also K3.COM
- net GND: now also Q3.3 (S)
- net NC: now also K3.NC
- net NO: now also K3.NO
- net Signal: now also Q3.2 (G)
- new net: D5.2 (A), K3.COIL2, Q3.1 (D)
- new net +12V: D5.1 (K), K3.COIL1

Commit message: Most of the layout completed
Parts:
- renumbered D5 to D7, K3 to K4, Q3 to Q5
Changed lines of the file:
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@@
 		(dnp no)
 		(fields_autoplaced yes)
-		(property "Reference" "D5"
+		(property "Reference" "D7"
 			(at 140.97 86.3599 90)
 			(effects
@@
 			(project "twingo_aa"
 				(path "/40f6f48c-88df-4c09-997b-20b4a32eb379/9deacaa5-e565-41f9-9e7d-763b562d8e76"
-					(reference "D5")
+					(reference "D7")
 					(unit 1)
 				)
@@
 		(dnp no)
 		(fields_autoplaced yes)
-		(property "Reference" "#PWR16"
+		(property "Reference" "#PWR045"
 			(at 138.43 118.11 0)
 			(effects
@@
 			(project "twingo_aa"
 				(path "/40f6f48c-88df-4c09-997b-20b4a32eb379/9deacaa5-e565-41f9-9e7d-763b562d8e76"
-					(reference "#PWR16")
+					(reference "#PWR045")
 					(unit 1)
 				)
@@
 		(dnp no)
 		(fields_autoplaced yes)
-		(property "Reference" "K3"
+		(property "Reference" "K4"
 			(at 158.75 73.66 0)
 			(effects
@@
 			(project "twingo_aa"
 				(path "/40f6f48c-88df-4c09-997b-20b4a32eb379/9deacaa5-e565-41f9-9e7d-763b562d8e76"
-					(reference "K3")
+					(reference "K4")
 					(unit 1)
 				)
@@
 		(dnp no)
 		(fields_autoplaced yes)
-		(property "Reference" "#PWR3"
+		(property "Reference" "#PWR044"
 			(at 138.43 85.09 0)
 			(effects
@@
 			(project "twingo_aa"
 				(path "/40f6f48c-88df-4c09-997b-20b4a32eb379/9deacaa5-e565-41f9-9e7d-763b562d8e76"
-					(reference "#PWR3")
+					(reference "#PWR044")
 					(unit 1)
 				)
@@
 		(dnp no)
 		(fields_autoplaced yes)
-		(property "Reference" "Q3"
+		(property "Reference" "Q5"
 			(at 142.24 102.8699 0)
 			(effects
@@
 			(project "twingo_aa"
 				(path "/40f6f48c-88df-4c09-997b-20b4a32eb379/9deacaa5-e565-41f9-9e7d-763b562d8e76"
-					(reference "Q3")
+					(reference "Q5")
 					(unit 1)
 				)
