File: 12v_to_5v.kicad_sch (KiCad schematic)
At the start: 15 parts, among them U3 TPS562210ADDFR

Commit message: Various fixes
Signed-off-by: Tobias de Bruijn <t.debruijn@array21.dev>
Parts:
- removed R14: 10K, symbol Device:R
- L1: footprint (none) -> footprints:TPS562210A_N
- R10, R9: footprint (none) -> Resistor_SMD:R_1206_3216Metric
- R11: value 304K -> 300K; footprint (none) -> Resistor_SMD:R_0603_1608Metric
- R12: footprint (none) -> Resistor_SMD:R_0402_1005Metric
- U3: footprint DDF0008A_N -> footprints:TPS562210A_N
Other:
- note added: "Should be 304K"
Changed lines of the file:
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@@
 (kicad_sch
-	(version 20231120)
+	(version 20250114)
 	(generator "eeschema")
-	(generator_version "8.0")
+	(generator_version "9.0")
 	(paper "A4")
+	(text "Should be 304K"
+		(exclude_from_sim no)
+		(at 257.048 86.36 0)
+		(effects
+			(font
+				(size 1.27 1.27)
+			)
+		)
+	)
 	(junction
 		(at 187.96 88.9)
@@
 	)
 	(junction
-		(at 254 76.2)
-		(diameter 0)
-		(color 0 0 0 0)
-	)
-	(junction
 		(at 180.34 76.2)
 		(diameter 0)
@@
 	)
 	(junction
-		(at 187.96 104.14)
-		(diameter 0)
-		(color 0 0 0 0)
-	)
-	(junction
 		(at 78.74 76.2)
 		(diameter 0)
@@
 	(wire
 		(pts
-			(xy 187.96 88.9) (xy 187.96 104.14)
+			(xy 187.96 88.9) (xy 187.96 107.95)
 		)
 		(stroke
@@
 	(wire
 		(pts
-			(xy 187.96 104.14) (xy 187.96 107.95)
-		)
-		(stroke
-			(width 0)
-			(type default)
-		)
-	)
-	(wire
-		(pts
-			(xy 195.58 104.14) (xy 254 104.14)
-		)
-		(stroke
-			(width 0)
-			(type default)
-		)
-	)
-	(wire
-		(pts
 			(xy 187.96 76.2) (xy 203.2 76.2)
 		)
@@
 	(wire
 		(pts
-			(xy 240.03 76.2) (xy 254 76.2)
+			(xy 240.03 76.2) (xy 257.81 76.2)
 		)
 		(stroke
@@
 	(wire
 		(pts
-			(xy 254 76.2) (xy 257.81 76.2)
-		)
-		(stroke
-			(width 0)
-			(type default)
-		)
-	)
-	(wire
-		(pts
 			(xy 66.04 76.2) (xy 78.74 76.2)
 		)
@@
 		(pts
 			(xy 203.2 83.82) (xy 214.63 83.82)
-		)
-		(stroke
-			(width 0)
-			(type default)
-		)
-	)
-	(wire
-		(pts
-			(xy 254 104.14) (xy 254 76.2)
 		)
 		(stroke
@@
 			)
 		)
-		(property "Footprint" ""
+		(property "Footprint" "Resistor_SMD:R_1206_3216Metric"
 			(at 186.182 85.09 90)
 			(effects
@@
 			)
 		)
-		(property "Footprint" ""
+		(property "Footprint" "footprints:TPS562210A_N"
 			(at 184.15 76.2 0)
 			(effects
@@
 			)
 		)
-		(property "Footprint" ""
+		(property "Footprint" "Resistor_SMD:R_0402_1005Metric"
 			(at 238.252 92.71 90)
 			(effects
@@
 			)
 		)
-		(property "Footprint" ""
+		(property "Footprint" "Resistor_SMD:R_1206_3216Metric"
 			(at 111.252 87.63 90)
 			(effects
@@
 			)
 		)
-		(property "Footprint" "DDF0008A_N"
+		(property "Footprint" "footprints:TPS562210A_N"
 			(at 149.86 86.36 0)
 			(effects
@@
 	(symbol
 		(lib_id "Device:R")
-		(at 191.77 104.14 90)
-		(unit 1)
-		(exclude_from_sim no)
-		(in_bom yes)
-		(on_board yes)
-		(dnp no)
-		(fields_autoplaced yes)
-		(property "Reference" "R14"
-			(at 191.77 97.79 90)
-			(effects
-				(font
-					(size 1.27 1.27)
-				)
-			)
-		)
-		(property "Value" "10K"
-			(at 191.77 100.33 90)
-			(effects
-				(font
-					(size 1.27 1.27)
-				)
-			)
-		)
-		(property "Footprint" ""
-			(at 191.77 105.918 90)
-			(effects
-				(font
-					(size 1.27 1.27)
-				)
-				(hide yes)
-			)
-		)
-		(property "Datasheet" "~"
-			(at 191.77 104.14 0)
-			(effects
-				(font
-					(size 1.27 1.27)
-				)
-				(hide yes)
-			)
-		)
-		(property "Description" "Resistor"
-			(at 191.77 104.14 0)
-			(effects
-				(font
-					(size 1.27 1.27)
-				)
-				(hide yes)
-			)
-		)
-		(pin "1"
-		)
-		(pin "2"
-		)
-		(instances
-			(project ""
-				(path "/40f6f48c-88df-4c09-997b-20b4a32eb379/e70bba1a-d775-4d26-a9ad-f32d1f28b359"
-					(reference "R14")
-					(unit 1)
-				)
-			)
-		)
-	)
-	(symbol
-		(lib_id "Device:R")
 		(at 240.03 85.09 0)
 		(unit 1)
@@
 			)
 		)
-		(property "Value" "304K"
+		(property "Value" "300K"
 			(at 242.57 86.3599 0)
 			(effects
@@
 			)
 		)
-		(property "Footprint" ""
+		(property "Footprint" "Resistor_SMD:R_0603_1608Metric"
 			(at 238.252 85.09 90)
 			(effects

Commit message: Most of the layout completed
Parts:
- L1: footprint footprints:TPS562210A_N -> Inductor_SMD:L_1206_3216Metric
- renumbered C11 to C10, C14 to C11, C15 to C12, C16 to C13, C12 to C14, C13 to C7, C9 to C8, C10 to C9, R11 to R10, R9 to R11, R10 to R9, U3 to U2
Changed lines of the file:
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@@
 	)
 	(symbol
+		(lib_name "GND_5")
 		(lib_id "power:GND")
 		(at 240.03 96.52 0)
@@
 		(dnp no)
 		(fields_autoplaced yes)
-		(property "Reference" "#PWR42"
+		(property "Reference" "#PWR037"
 			(at 240.03 102.87 0)
 			(effects
@@
 			(project ""
 				(path "/40f6f48c-88df-4c09-997b-20b4a32eb379/e70bba1a-d775-4d26-a9ad-f32d1f28b359"
-					(reference "#PWR42")
+					(reference "#PWR037")
 					(unit 1)
 				)
@@
 		(dnp no)
 		(fields_autoplaced yes)
-		(property "Reference" "C16"
+		(property "Reference" "C13"
 			(at 231.14 78.7399 0)
 			(effects
@@
 			(project "twingo_aa"
 				(path "/40f6f48c-88df-4c09-997b-20b4a32eb379/e70bba1a-d775-4d26-a9ad-f32d1f28b359"
-					(reference "C16")
+					(reference "C13")
 					(unit 1)
 				)
@@
 		(dnp no)
 		(fields_autoplaced yes)
-		(property "Reference" "#PWR40"
+		(property "Reference" "#PWR038"
 			(at 172.72 105.41 0)
 			(effects
@@
 			(project "twingo_aa"
 				(path "/40f6f48c-88df-4c09-997b-20b4a32eb379/e70bba1a-d775-4d26-a9ad-f32d1f28b359"
-					(reference "#PWR40")
+					(reference "#PWR038")
 					(unit 1)
 				)
@@
 		(dnp no)
 		(fields_autoplaced yes)
-		(property "Reference" "C10"
+		(property "Reference" "C9"
 			(at 82.55 78.7399 0)
 			(effects
@@
 			(project "twingo_aa"
 				(path "/40f6f48c-88df-4c09-997b-20b4a32eb379/e70bba1a-d775-4d26-a9ad-f32d1f28b359"
-					(reference "C10")
-					(unit 1)
-				)
-			)
-		)
-	)
-	(symbol
+					(reference "C9")
+					(unit 1)
+				)
+			)
+		)
+	)
+	(symbol
+		(lib_name "GND_2")
 		(lib_id "power:GND")
 		(at 120.65 101.6 0)
@@
 		(dnp no)
 		(fields_autoplaced yes)
-		(property "Reference" "#PWR39"
+		(property "Reference" "#PWR039"
 			(at 120.65 107.95 0)
 			(effects
@@
 			(project "twingo_aa"
 				(path "/40f6f48c-88df-4c09-997b-20b4a32eb379/e70bba1a-d775-4d26-a9ad-f32d1f28b359"
-					(reference "#PWR39")
+					(reference "#PWR039")
 					(unit 1)
 				)
@@
 		(dnp no)
 		(fields_autoplaced yes)
-		(property "Reference" "R10"
+		(property "Reference" "R9"
 			(at 190.5 83.8199 0)
 			(effects
@@
 			(project ""
 				(path "/40f6f48c-88df-4c09-997b-20b4a32eb379/e70bba1a-d775-4d26-a9ad-f32d1f28b359"
-					(reference "R10")
+					(reference "R9")
 					(unit 1)
 				)
@@
 		(dnp no)
 		(fields_autoplaced yes)
-		(property "Reference" "C15"
+		(property "Reference" "C12"
 			(at 218.44 78.7399 0)
 			(effects
@@
 			(project "twingo_aa"
 				(path "/40f6f48c-88df-4c09-997b-20b4a32eb379/e70bba1a-d775-4d26-a9ad-f32d1f28b359"
-					(reference "C15")
+					(reference "C12")
 					(unit 1)
 				)
@@
 			)
 		)
-		(property "Footprint" "footprints:TPS562210A_N"
+		(property "Footprint" "Inductor_SMD:L_1206_3216Metric"
 			(at 184.15 76.2 0)
 			(effects
@@
 		(dnp no)
 		(fields_autoplaced yes)
-		(property "Reference" "C11"
+		(property "Reference" "C10"
 			(at 93.98 78.7399 0)
 			(effects
@@
 			(project "twingo_aa"
 				(path "/40f6f48c-88df-4c09-997b-20b4a32eb379/e70bba1a-d775-4d26-a9ad-f32d1f28b359"
-					(reference "C11")
+					(reference "C10")
 					(unit 1)
 				)
@@
 		(dnp no)
 		(fields_autoplaced yes)
-		(property "Reference" "C13"
+		(property "Reference" "C7"
 			(at 176.53 68.58 90)
 			(effects
@@
 			(project ""
 				(path "/40f6f48c-88df-4c09-997b-20b4a32eb379/e70bba1a-d775-4d26-a9ad-f32d1f28b359"
-					(reference "C13")
+					(reference "C7")
 					(unit 1)
 				)
@@
 		(dnp no)
 		(fields_autoplaced yes)
-		(property "Reference" "R9"
+		(property "Reference" "R11"
 			(at 115.57 86.3599 0)
 			(effects
@@
 			(project ""
 				(path "/40f6f48c-88df-4c09-997b-20b4a32eb379/e70bba1a-d775-4d26-a9ad-f32d1f28b359"
-					(reference "R9")
+					(reference "R11")
 					(unit 1)
 				)
@@
 		(dnp no)
 		(fields_autoplaced yes)
-		(property "Reference" "U3"
+		(property "Reference" "U2"
 			(at 149.86 66.04 0)
 			(effects
@@
 			(project ""
 				(path "/40f6f48c-88df-4c09-997b-20b4a32eb379/e70bba1a-d775-4d26-a9ad-f32d1f28b359"
-					(reference "U3")
+					(reference "U2")
 					(unit 1)
 				)
@@
 		(dnp no)
 		(fields_autoplaced yes)
-		(property "Reference" "R11"
+		(property "Reference" "R10"
 			(at 242.57 83.8199 0)
 			(effects
@@
 			(project "twingo_aa"
 				(path "/40f6f48c-88df-4c09-997b-20b4a32eb379/e70bba1a-d775-4d26-a9ad-f32d1f28b359"
-					(reference "R11")
-					(unit 1)
-				)
-			)
-		)
-	)
-	(symbol
+					(reference "R10")
+					(unit 1)
+				)
+			)
+		)
+	)
+	(symbol
+		(lib_name "GND_1")
 		(lib_id "power:GND")
 		(at 113.03 91.44 0)
@@
 		(dnp no)
 		(fields_autoplaced yes)
-		(property "Reference" "#PWR38"
+		(property "Reference" "#PWR036"
 			(at 113.03 97.79 0)
 			(effects
@@
 			(project "twingo_aa"
 				(path "/40f6f48c-88df-4c09-997b-20b4a32eb379/e70bba1a-d775-4d26-a9ad-f32d1f28b359"
-					(reference "#PWR38")
+					(reference "#PWR036")
 					(unit 1)
 				)
@@
 		(dnp no)
 		(fields_autoplaced yes)
-		(property "Reference" "C14"
+		(property "Reference" "C11"
 			(at 207.01 78.7399 0)
 			(effects
@@
 			(project ""
 				(path "/40f6f48c-88df-4c09-997b-20b4a32eb379/e70bba1a-d775-4d26-a9ad-f32d1f28b359"
-					(reference "C14")
+					(reference "C11")
 					(unit 1)
 				)
@@
 		(dnp no)
 		(fields_autoplaced yes)
-		(property "Reference" "C9"
+		(property "Reference" "C8"
 			(at 69.85 78.7399 0)
 			(effects
@@
 			(project ""
 				(path "/40f6f48c-88df-4c09-997b-20b4a32eb379/e70bba1a-d775-4d26-a9ad-f32d1f28b359"
-					(reference "C9")
+					(reference "C8")
 					(unit 1)
 				)
@@
 		(dnp no)
 		(fields_autoplaced yes)
-		(property "Reference" "C12"
+		(property "Reference" "C14"
 			(at 124.46 96.5199 0)
 			(effects
@@
 			(project ""
 				(path "/40f6f48c-88df-4c09-997b-20b4a32eb379/e70bba1a-d775-4d26-a9ad-f32d1f28b359"
-					(reference "C12")
-					(unit 1)
-				)
-			)
-		)
-	)
-	(symbol
+					(reference "C14")
+					(unit 1)
+				)
+			)
+		)
+	)
+	(symbol
+		(lib_name "GND_3")
 		(lib_id "power:GND")
 		(at 66.04 83.82 0)
@@
 		(dnp no)
 		(fields_autoplaced yes)
-		(property "Reference" "#PWR37"
+		(property "Reference" "#PWR034"
 			(at 66.04 90.17 0)
 			(effects
@@
 			(project ""
 				(path "/40f6f48c-88df-4c09-997b-20b4a32eb379/e70bba1a-d775-4d26-a9ad-f32d1f28b359"
-					(reference "#PWR37")
-					(unit 1)
-				)
-			)
-		)
-	)
-	(symbol
+					(reference "#PWR034")
+					(unit 1)
+				)
+			)
+		)
+	)
+	(symbol
+		(lib_name "GND_4")
 		(lib_id "power:GND")
 		(at 203.2 83.82 0)
@@
 		(dnp no)
 		(fields_autoplaced yes)
-		(property "Reference" "#PWR41"
+		(property "Reference" "#PWR035"
 			(at 203.2 90.17 0)
 			(effects
@@
 			(project "twingo_aa"
 				(path "/40f6f48c-88df-4c09-997b-20b4a32eb379/e70bba1a-d775-4d26-a9ad-f32d1f28b359"
-					(reference "#PWR41")
-					(unit 1)
-				)
+					(reference "#PWR035")
+					(unit 1)
+				)
