File: 3v_switched_relay.kicad_sch (KiCad schematic)
At the start: 4 parts, among them K1 SRD-05VDC-SL-C, Q1 BS170

Commit message: Most of the layout completed
Parts:
- K1: footprint footprints:SRD-05VDC-SL-C -> footprints:RELAY_SRD-05VDC-SL-C
- renumbered D3 to D4
Changed lines of the file:
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@@
 			)
 		)
-		(property "Footprint" "footprints:SRD-05VDC-SL-C"
+		(property "Footprint" "footprints:RELAY_SRD-05VDC-SL-C"
 			(at 146.05 95.25 0)
 			(effects
@@
 		(dnp no)
 		(fields_autoplaced yes)
-		(property "Reference" "#PWR2"
+		(property "Reference" "#PWR029"
 			(at 130.81 129.54 0)
 			(effects
@@
 			(project "twingo_aa"
 				(path "/40f6f48c-88df-4c09-997b-20b4a32eb379/7b2498f2-a50b-4ca1-aa81-485de40240be"
-					(reference "#PWR25")
+					(reference "#PWR031")
 					(unit 1)
 				)
 				(path "/40f6f48c-88df-4c09-997b-20b4a32eb379/c1c62b4b-e08e-4f46-8e45-465316d28a17"
-					(reference "#PWR2")
+					(reference "#PWR029")
 					(unit 1)
 				)
@@
 		(on_board yes)
 		(dnp no)
-		(property "Reference" "D3"
+		(property "Reference" "D4"
 			(at 128.27 95.2499 90)
 			(effects
@@
 			(project "twingo_aa"
 				(path "/40f6f48c-88df-4c09-997b-20b4a32eb379/7b2498f2-a50b-4ca1-aa81-485de40240be"
+					(reference "D5")
+					(unit 1)
+				)
+				(path "/40f6f48c-88df-4c09-997b-20b4a32eb379/c1c62b4b-e08e-4f46-8e45-465316d28a17"
 					(reference "D4")
-					(unit 1)
-				)
-				(path "/40f6f48c-88df-4c09-997b-20b4a32eb379/c1c62b4b-e08e-4f46-8e45-465316d28a17"
-					(reference "D3")
 					(unit 1)
 				)
@@
 			(project ""
 				(path "/40f6f48c-88df-4c09-997b-20b4a32eb379/7b2498f2-a50b-4ca1-aa81-485de40240be"
-					(reference "R13")
+					(reference "R7")
 					(unit 1)
 				)
@@
 		(dnp no)
 		(fields_autoplaced yes)
-		(property "Reference" "#PWR101"
+		(property "Reference" "#PWR028"
 			(at 130.81 96.52 0)
 			(effects
@@
 			(project "twingo_aa"
 				(path "/40f6f48c-88df-4c09-997b-20b4a32eb379/7b2498f2-a50b-4ca1-aa81-485de40240be"
-					(reference "#PWR4")
+					(reference "#PWR030")
 					(unit 1)
 				)
 				(path "/40f6f48c-88df-4c09-997b-20b4a32eb379/c1c62b4b-e08e-4f46-8e45-465316d28a17"
-					(reference "#PWR101")
-					(unit 1)
-				)
+					(reference "#PWR028")
+					(unit 1)
+				)
