File: 5v_to_3v3.kicad_sch (KiCad schematic)
At the start: 3 parts, among them U1 XC6206PxxxMR

Commit message: Most of the layout completed
Parts:
- renumbered C7 to C15, C8 to C16, U1 to U3
Changed lines of the file:
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@@
 	)
 	(symbol
+		(lib_name "GND_2")
 		(lib_id "power:GND")
 		(at 146.05 90.17 0)
@@
 		(dnp no)
 		(fields_autoplaced yes)
-		(property "Reference" "#PWR35"
+		(property "Reference" "#PWR041"
 			(at 146.05 96.52 0)
 			(effects
@@
 			(project "twingo_aa"
 				(path "/40f6f48c-88df-4c09-997b-20b4a32eb379/e76bedfd-b1e9-4b7f-8658-1c8889c6a913"
-					(reference "#PWR35")
+					(reference "#PWR041")
 					(unit 1)
 				)
@@
 		(dnp no)
 		(fields_autoplaced yes)
-		(property "Reference" "U1"
+		(property "Reference" "U3"
 			(at 146.05 76.2 0)
 			(effects
@@
 			(project ""
 				(path "/40f6f48c-88df-4c09-997b-20b4a32eb379/e76bedfd-b1e9-4b7f-8658-1c8889c6a913"
-					(reference "U1")
-					(unit 1)
-				)
-			)
-		)
-	)
-	(symbol
+					(reference "U3")
+					(unit 1)
+				)
+			)
+		)
+	)
+	(symbol
+		(lib_name "GND_1")
 		(lib_id "power:GND")
 		(at 127 90.17 0)
@@
 		(dnp no)
 		(fields_autoplaced yes)
-		(property "Reference" "#PWR34"
+		(property "Reference" "#PWR040"
 			(at 127 96.52 0)
 			(effects
@@
 			(project ""
 				(path "/40f6f48c-88df-4c09-997b-20b4a32eb379/e76bedfd-b1e9-4b7f-8658-1c8889c6a913"
-					(reference "#PWR34")
+					(reference "#PWR040")
 					(unit 1)
 				)
@@
 		(dnp no)
 		(fields_autoplaced yes)
-		(property "Reference" "#PWR36"
+		(property "Reference" "#PWR042"
 			(at 163.83 96.52 0)
 			(effects
@@
 			(project "twingo_aa"
 				(path "/40f6f48c-88df-4c09-997b-20b4a32eb379/e76bedfd-b1e9-4b7f-8658-1c8889c6a913"
-					(reference "#PWR36")
+					(reference "#PWR042")
 					(unit 1)
 				)
@@
 		(dnp no)
 		(fields_autoplaced yes)
-		(property "Reference" "C7"
+		(property "Reference" "C15"
 			(at 130.81 85.0899 0)
 			(effects
@@
 			(project ""
 				(path "/40f6f48c-88df-4c09-997b-20b4a32eb379/e76bedfd-b1e9-4b7f-8658-1c8889c6a913"
-					(reference "C7")
+					(reference "C15")
 					(unit 1)
 				)
@@
 		(dnp no)
 		(fields_autoplaced yes)
-		(property "Reference" "C8"
+		(property "Reference" "C16"
 			(at 167.64 85.0899 0)
 			(effects
@@
 			(project "twingo_aa"
 				(path "/40f6f48c-88df-4c09-997b-20b4a32eb379/e76bedfd-b1e9-4b7f-8658-1c8889c6a913"
-					(reference "C8")
-					(unit 1)
-				)
+					(reference "C16")
+					(unit 1)
+				)
