File: twingo_aa.kicad_pcb (KiCad board)
At the start: 4 copper layers, 56.3 x 65 mm, 48 parts, among them J1 Conn_01x02_Male 3.3v power, J2 Conn_01x02_Male USB power MAX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, J3 Conn_01x06_Male DEBUG, J4 Conn_02x20_RPI, Q1 BS170, Q2 BS170, Q3 BS170, Q4 BS170, Q5 BS170, U1 XC6206PxxxMR, U2 STM32L151CBTxA

Commit message: Various fixes
Signed-off-by: Tobias de Bruijn <t.debruijn@array21.dev>
Parts:
- removed G*** (x2): LOGO, LOGO
- removed J1: Conn_01x02_Male 3.3v power, Connector_PinHeader_2.54mm:PinHeader_1x02_P2.54mm_Vertical
- removed J2: Conn_01x02_Male USB power MAX 7v, Connector_PinHeader_2.54mm:PinHeader_1x02_P2.54mm_Vertical
- removed R1: 1K8, Resistor_SMD:R_0603_1608Metric
- removed S1: TS-1187A-B-A-B, Mr_Friendly_SmartPCB:TS1187ABAB
- added D5: 1N4007, Diode_THT:D_DO-41_SOD81_P10.16mm_Horizontal, F.Cu at (25.9, 44.9)
- added J5: Screw_Terminal_01x04, TerminalBlock:TerminalBlock_bornier-4_P5.08mm, F.Cu at (158.5, 121.0)
- added J6: Screw_Terminal_01x06, TerminalBlock:TerminalBlock_bornier-6_P5.08mm, F.Cu at (121.8, 64.0)
- added K1: SRD-05VDC-SL-C, footprints:SRD-05VDC-SL-C, F.Cu at (113.8, 77.5)
- added K2: SRD-05VDC-SL-C, footprints:SRD-05VDC-SL-C, F.Cu at (113.8, 93.5)
- added K3: SRD-12VDC-SL-C, footprints:RELAY_SRD-12VDC-SL-C, F.Cu at (122.0, 110.0)
- added K4: SRD-12VDC-SL-C, footprints:RELAY_SRD-12VDC-SL-C, F.Cu at (150.5, 108.5)
- added L1: 4.7uH, footprints:TPS562210A_N, F.Cu at (72.6, 50.3)
- added Q3: BS170, Package_TO_SOT_THT:TO-92_Inline, F.Cu at (40.0, 46.0)
- added Q6: BS170, Package_TO_SOT_THT:TO-92_Inline, F.Cu at (65.6, 8.68)
- added R10: 100K, Resistor_SMD:R_1206_3216Metric, F.Cu at (78.0, 53.0)
- added R11: 300K, Resistor_SMD:R_0603_1608Metric, F.Cu at (77.2, 55.9)
- added R12: 54.9K, Resistor_SMD:R_0402_1005Metric, F.Cu at (76.7, 58.1)
- added R13: 10K, Resistor_SMD:R_1206_3216Metric, F.Cu at (50.4, 66.5)
- added R14: 100K, Resistor_SMD:R_1206_3216Metric, F.Cu at (60.8, 7.07)
- added R16: 0.75K, Resistor_SMD:R_0805_2012Metric, F.Cu at (51.1, 15.9)
- added R17: 100K, Resistor_SMD:R_1206_3216Metric, F.Cu at (60.8, 10.4)
- added R6: 10K, Resistor_SMD:R_1206_3216Metric, F.Cu at (26.9, 69.0)
- added R8: 10K, Resistor_SMD:R_1206_3216Metric, F.Cu at (50.4, 44.4)
- added R9: 10K, Resistor_SMD:R_1206_3216Metric, F.Cu at (78.0, 49.7)
- added TP1: TestPoint, TestPoint:TestPoint_Pad_D1.0mm, F.Cu at (47.3, 16.0)
- added TP2: TestPoint, TestPoint:TestPoint_Pad_D1.0mm, F.Cu at (47.3, 19.1)
- added TP3: TestPoint, TestPoint:TestPoint_Pad_D1.0mm, F.Cu at (47.3, 22.1)
- added U3: TPS562210ADDFR, footprints:TPS562210A_N, F.Cu at (156.0, 88.7)
- U1: moved to F.Cu
- moved C1 75.7 mm to (88.4, 40.1), turned to 0 degrees
- moved D5 74.9 mm to (133.5, 114.7), turned to 90 degrees
- moved Q3 74.3 mm to (137.5, 112.0), turned to -90 degrees
- moved Q4 73.8 mm to (138.5, 120.5), turned to 180 degrees
- moved D6 73.5 mm to (142.9, 98.5)
- moved C2 63.0 mm to (88.4, 43.1), turned to 0 degrees
- moved C5 60.9 mm to (88.4, 52.1), turned to 0 degrees
- moved C3 58.1 mm to (88.4, 46.1)
- moved C4 56.8 mm to (88.4, 49.1), turned to 0 degrees
- moved C6 55.9 mm to (88.4, 55.1)
- moved R4 52.8 mm to (92.7, 56.2)
- moved U1 51.2 mm to (88.8, 61.9), turned to 0 degrees
- moved D7 49.5 mm to (134.0, 99.7), turned to 90 degrees
- moved R3 44.8 mm to (92.7, 53.7), turned to 0 degrees
- moved R5 41.9 mm to (101.9, 51.6)
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Connections:
- C14 pad 2: /12v_to_5v/5V -> /12v_switched_relay_no_pulldown/Signal
- C15 pad 2: /12v_to_5v/5V -> /12v_switched_relay_no_pulldown/Signal
- C16 pad 2: /12v_to_5v/5V -> /12v_switched_relay_no_pulldown/Signal
Routing:
- net (no net): track 65.5 -> 7.01 mm, vias 2 -> 0
- net Net-(D6-A): track 0.00 -> 37.1 mm
- net DEBUG_TX: track 33.7 -> 0.00 mm, vias 2 -> 0
- net DEBUG_RX: track 33.2 -> 0.00 mm, vias 2 -> 0
- net PI_TX: track 32.6 -> 0.00 mm
- net PI_RX: track 29.6 -> 0.00 mm
- net DEBUG_SWDIO: track 28.6 -> 0.00 mm
- net +3.3V: track 28.5 -> 0.00 mm, vias 7 -> 0
- net GND: track 28.3 -> 0.00 mm, vias 17 -> 0
- net DEBUG_SWCLK: track 27.2 -> 0.00 mm
- net unconnected-(U2-PB2-Pad20): track 23.0 -> 0.00 mm, vias 3 -> 0
- net RFM69_RESET: track 20.2 -> 0.00 mm, vias 1 -> 0
- net DEBUG_LED: track 18.9 -> 0.00 mm, vias 2 -> 0
- net DEBUG_LED_2: track 18.5 -> 0.00 mm, vias 2 -> 0
- net Car_12V: track 0.00 -> 16.3 mm
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Other:
- board text removed: "3.3v"

Commit message: Most of the layout completed
Parts:
- removed the D5 at (133.5, 114.7)
- removed the D5 at (25.9, 44.9)
- removed D8, D9: LED, LED_SMD:LED_0805_2012Metric
- removed J5: Screw_Terminal_01x04, TerminalBlock:TerminalBlock_bornier-4_P5.08mm
- removed J6: Screw_Terminal_01x06, TerminalBlock:TerminalBlock_bornier-6_P5.08mm
- removed the Q3 at (40.0, 46.0)
- removed the Q3 at (137.5, 112.0)
- removed Q6: BS170, Package_TO_SOT_THT:TO-92_Inline
- removed R16: 0.75K, Resistor_SMD:R_0805_2012Metric
- removed R17: 100K, Resistor_SMD:R_1206_3216Metric
- added D5: 1N4007, Diode_THT:D_DO-41_SOD81_P10.16mm_Horizontal, F.Cu at (139.1, 82.5)
- added J1: Conn_01x06_Male DEBUG, Connector_JST:JST_SHL_SM06B-SHLS-TF_1x06-1MP_P1.00mm_Horizontal, F.Cu at (107.2, 62.6)
- added J2: Conn_02x20_RPI, Connector_PinSocket_2.54mm:PinSocket_2x20_P2.54mm_Vertical, B.Cu at (163.1, 68.1)
- added Q3: BS170, Package_TO_SOT_THT:TO-92_Inline, F.Cu at (157.5, 94.3)
- added R1: 10K, Resistor_SMD:R_1206_3216Metric, F.Cu at (103.5, 67.3)
- added R7: 10K, Resistor_SMD:R_1206_3216Metric, F.Cu at (130.2, 94.0)
- added S2: TS-1187A-B-A-B, footprints:SW_TS-1187A-B-A-B, F.Cu at (92.0, 72.8)
- C11: value 10uF -> 22uF
- C12: value 8200pF -> 22uF; footprint Capacitor_SMD:C_0603_1608Metric -> Capacitor_SMD:C_1206_3216Metric
- C13: value 100nF -> 22uF; footprint Capacitor_SMD:C_0402_1005Metric -> Capacitor_SMD:C_1206_3216Metric
- C14: value 22uF -> 8200pF; footprint Capacitor_SMD:C_1206_3216Metric -> Capacitor_SMD:C_0603_1608Metric
- C15, C16: value 22uF -> 1uF
- C7, C8: value 1uF -> 100nF; footprint Capacitor_SMD:C_1206_3216Metric -> Capacitor_SMD:C_0402_1005Metric
- C9: value 100nF -> 10uF; footprint Capacitor_SMD:C_0402_1005Metric -> Capacitor_SMD:C_1206_3216Metric
- D3: value 1N4007 -> LED; footprint Diode_THT:D_DO-41_SOD81_P10.16mm_Horizontal -> LED_SMD:LED_0805_2012Metric
- J3: value Conn_01x06_Male DEBUG -> Screw_Terminal_01x04; footprint Connector_JST:JST_SHL_SM06B-SHLS-TF_1x06-1MP_P1.00mm_Horizontal -> TerminalBlock:TerminalBlock_bornier-4_P5.08mm
- J4: value Conn_02x20_RPI -> Screw_Terminal_01x06; footprint Connector_PinSocket_2.54mm:PinSocket_2x20_P2.54mm_Vertical -> TerminalBlock:TerminalBlock_bornier-6_P5.08mm; moved to F.Cu
- K1, K2: footprint footprints:SRD-05VDC-SL-C -> footprints:RELAY_SRD-05VDC-SL-C
- L1: footprint footprints:TPS562210A_N -> Inductor_SMD:L_1206_3216Metric
- R10: value 100K -> 300K; footprint Resistor_SMD:R_1206_3216Metric -> Resistor_SMD:R_0603_1608Metric
- R11: value 300K -> 10K; footprint Resistor_SMD:R_0603_1608Metric -> Resistor_SMD:R_1206_3216Metric
- R13, R9: value 10K -> 100K
- R5: value 10K -> 0.75K; footprint Resistor_SMD:R_1206_3216Metric -> Resistor_SMD:R_0805_2012Metric
- U1: value XC6206PxxxMR -> STM32L151CBTxA; footprint Package_TO_SOT_SMD:SOT-23-3 -> Package_QFP:LQFP-48_7x7mm_P0.5mm
- U2: value STM32L151CBTxA -> TPS562210ADDFR; footprint Package_QFP:LQFP-48_7x7mm_P0.5mm -> footprints:TPS562210A_N
- U3: value TPS562210ADDFR -> XC6206PxxxMR; footprint footprints:TPS562210A_N -> Package_TO_SOT_SMD:SOT-23-3
- moved TP2 120.5 mm to (119.9, 115.3)
- moved R8 115.0 mm to (156.2, 89.5), turned to 90 degrees
- moved R6 114.1 mm to (139.1, 89.5), turned to 90 degrees
- moved TP1 107.8 mm to (112.3, 102.1)
- moved R14 95.5 mm to (86.4, 99.1)
- moved TP3 91.9 mm to (102.6, 95.5)
- moved J3 86.2 mm to (81.9, 106.0), turned to -90 degrees
- moved J4 81.4 mm to (81.9, 62.9), turned to -90 degrees
- moved C15 73.8 mm to (117.5, 92.1), turned to 90 degrees
- moved R9 72.1 mm to (96.5, 119.4)
- moved R11 71.1 mm to (110.5, 118.7), turned to -90 degrees
- moved Q1 70.4 mm to (140.3, 94.3), turned to 180 degrees
- moved U2 69.4 mm to (103.5, 116.2)
- moved C14 68.3 mm to (107.3, 119.4), turned to -90 degrees
- moved R10 68.0 mm to (109.2, 113.5), turned to -90 degrees
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Connections:
- C1 pad 1: +3.3V -> +3V3
- C11 pad 1: +12V -> GND
- C11 pad 2: GND -> /12v_switched_relay_no_pulldown/Com
- C12 pad 1: Net-(U3-SS) -> GND
- C12 pad 2: GND -> /12v_switched_relay_no_pulldown/Com
- C13 pad 1: Net-(U3-VBST) -> GND
- C13 pad 2: Net-(U3-SW) -> /12v_switched_relay_no_pulldown/Com
- C14 pad 1: GND -> Net-(U2-SS)
- C14 pad 2: /12v_switched_relay_no_pulldown/Signal -> GND
- C15 pad 1: GND -> +5V
- C15 pad 2: /12v_switched_relay_no_pulldown/Signal -> GND
- C16 pad 1: GND -> +3V3
- C16 pad 2: /12v_switched_relay_no_pulldown/Signal -> GND
- C2 pad 1: +3.3V -> +3V3
- C3 pad 1: +3.3V -> +3V3
- C4 pad 1: +3.3V -> +3V3
- C5 pad 1: +3.3V -> +3V3
- C6 pad 1: +3.3V -> +3V3
- C7 pad 1: +5V -> Net-(U2-VBST)
- C7 pad 2: GND -> Net-(U2-SW)
- C8 pad 1: +3V3 -> +12V
- D3 pad 1: +5V -> Net-(D3-K)
- D3 pad 2: Net-(D3-A) -> +5V
- D7 pad 1: +5V -> +12V
- J3 pad 1: GND -> Car_12V
- J3 pad 2: +3.3V -> Amplifier_Enable_12V
- J3 pad 3: DEBUG_SWCLK -> Car_Remote_12V
- J3 pad 4: DEBUG_SWDIO -> GND
- J4 pad 1: +3.3V -> Car_Steering_Black
- J4 pad 2: +5V -> Car_Steering_Blue
- J4 pad 3: unconnected-(J4-Pin_3-Pad3) -> Car_Steering_Red
- J4 pad 4: +5V -> Car_Steering_Green
- J4 pad 5: unconnected-(J4-Pin_5-Pad5) -> Car_Steering_Yellow
- J4 pad 6: GND -> Car_Steering_Brown
- K3 pad COIL2: Net-(D5-A) -> Net-(D6-A)
- K3 pad COM: /12v_switched_relay_no_pulldown/Com -> Car_12V
- K3 pad NC: +5V -> /12v_switched_relay1/NC
- K3 pad NO: /12v_switched_relay_no_pulldown/NO -> +12V
- K4 pad COIL2: Net-(D6-A) -> Net-(D7-A)
- K4 pad COM: Car_12V -> /12v_switched_relay_no_pulldown/Com
- K4 pad NC: /12v_switched_relay1/NC -> +5V
- K4 pad NO: +12V -> /12v_switched_relay_no_pulldown/NO
- L1 pad 1: Net-(U3-SW) -> Net-(U2-SW)
- L1 pad 2: /12v_switched_relay_no_pulldown/Signal -> /12v_switched_relay_no_pulldown/Com
- Q1 pad 1: Net-(D3-A) -> Net-(D4-A)
- Q2 pad 1: Net-(D4-A) -> Net-(D5-A)
- Q4 pad 1: Net-(D6-A) -> Car_Remote
- Q5 pad 2: /12v_to_5v/Power Good -> /12v_switched_relay_no_pulldown/Signal
- R10 pad 1: /12v_switched_relay_no_pulldown/Signal -> /12v_switched_relay_no_pulldown/Com
- R10 pad 2: /12v_switched_relay_no_pulldown/Com -> Net-(U2-VFB)
- R11 pad 1: /12v_switched_relay_no_pulldown/Signal -> +12V
- R11 pad 2: Net-(U3-VFB) -> GND
- R12 pad 1: Net-(U3-VFB) -> Net-(U2-VFB)
- R13 pad 1: Amplifier_Enabled -> Car_Remote
- R13 pad 2: GND -> +3V3
- R14 pad 1: Car_Remote -> Car_Remote_12V
- R14 pad 2: +3V3 -> GND
- R4 pad 2: +3.3V -> +3V3
- R5 pad 2: Net-(U2-BOOT0) -> Net-(D3-K)
- R9 pad 1: +12V -> /12v_switched_relay_no_pulldown/Com
- R9 pad 2: GND -> /12v_switched_relay_no_pulldown/Signal
- TP1 pad 1: +3V3 -> +5V
- TP3 pad 1: +5V -> +3V3
- U1 pad 1: GND -> +3V3
- U1 pad 2: +3V3 -> unconnected-(U1-PC13-Pad2)
- U1 pad 3: +5V -> unconnected-(U1-PC14-Pad3)
- U2 pad 1: +3.3V -> GND
- U2 pad 2: unconnected-(U2-PC13-Pad2) -> Net-(U2-SW)
- U2 pad 3: unconnected-(U2-PC14-Pad3) -> +12V
- U2 pad 4: unconnected-(U2-PC15-Pad4) -> /12v_switched_relay_no_pulldown/Signal
- U2 pad 5: unconnected-(U2-PH0-Pad5) -> Net-(U2-SS)
- U2 pad 6: unconnected-(U2-PH1-Pad6) -> Net-(U2-VFB)
- U2 pad 7: STM32_RESET -> +12V
- U2 pad 8: GND -> Net-(U2-VBST)
- U3 pad 2: Net-(U3-SW) -> +3V3
- U3 pad 3: +12V -> +5V
Routing:
- net +12V: track 4.61 -> 206.1 mm, vias 0 -> 4
- net /12v_switched_relay_no_pulldown/Com: track 0.00 -> 158.3 mm, vias 0 -> 7
- net +5V: track 0.00 -> 144.6 mm, vias 0 -> 5
- net Car_Remote_12V: track 13.9 -> 111.6 mm, vias 0 -> 6
- net GND: track 0.00 -> 82.2 mm, vias 0 -> 30
- net Amplifier_Enable_12V: track 0.00 -> 81.1 mm, vias 0 -> 2
- net Car_12V: track 16.3 -> 90.7 mm, vias 0 -> 1
- net /12v_switched_relay_no_pulldown/Signal: track 0.00 -> 72.3 mm, vias 0 -> 4
- net Secondary_Power_Enable: track 0.00 -> 65.7 mm, vias 0 -> 2
- net PI_RX: track 0.00 -> 63.8 mm, vias 0 -> 2
- net PI_Vol_Down: track 0.00 -> 62.1 mm, vias 0 -> 1
- net PI_Vol_Up: track 0.00 -> 61.3 mm, vias 0 -> 1
- net PI_TX: track 0.00 -> 61.3 mm, vias 0 -> 1
- net PI_Track_Prev: track 0.00 -> 60.4 mm, vias 0 -> 1
- net PI_Track_Next: track 0.00 -> 59.5 mm, vias 0 -> 1
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- added copper zone on In2.Cu, net +3V3
- removed copper zone on In2.Cu, net +3.3V
Other:
- board size 56.3 x 65 mm -> 91.2 x 65 mm
- board text added: "5V OK"
- board text removed: "vcc"
