File: twingo_aa.kicad_sch (KiCad schematic)
At the start: 31 parts, among them J1 Conn_01x02_Male 3.3v power, J2 Conn_01x02_Male USB power MAX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, J3 Conn_01x06_Male DEBUG, J4 Conn_02x20_RPI, J5 Screw_Terminal_01x04, J6 Screw_Terminal_01x06, U2 STM32L151CBTxA

Commit message: Various fixes
Signed-off-by: Tobias de Bruijn <t.debruijn@array21.dev>
Parts:
- removed D8: LED, LED_SMD:LED_0805_2012Metric, symbol Device:LED
- removed J1: Conn_01x02_Male 3.3v power, Connector_PinHeader_2.54mm:PinHeader_1x02_P2.54mm_Vertical, symbol Connector:Conn_01x02_Male
- removed J2: Conn_01x02_Male USB power MAX 7v, Connector_PinHeader_2.54mm:PinHeader_1x02_P2.54mm_Vertical, symbol Connector:Conn_01x02_Male
- removed R15: 0.75K, symbol Device:R
- J5: footprint (none) -> TerminalBlock:TerminalBlock_bornier-4_P5.08mm
- J6: footprint (none) -> TerminalBlock:TerminalBlock_bornier-6_P5.08mm
- R16: footprint (none) -> Resistor_SMD:R_0805_2012Metric
- TP1, TP2, TP3: footprint (none) -> TestPoint:TestPoint_Pad_D1.0mm
Connections:
- net 12v_to_5v/5V renamed 12v_switched_relay_no_pulldown/Signal
- no-connect marks 39 -> 38
Other:
- removed sheet 12v_switched_relay
- removed sheet 3v_switched_relay2
- added sheet 12v_detect (12v_detect.kicad_sch)
- added sheet 12v_switched_relay_no_pulldown (12v_switched_relay_no_pulldown.kicad_sch)
- moved on the sheet: TP2

Commit message: Most of the layout completed
Parts:
- removed S1: TS-1187A-B-A-B, Mr_Friendly_SmartPCB:TS1187ABAB, symbol MrFriendly:TS-1187A-B-A-B
- added S2: TS-1187A-B-A-B, footprints:SW_TS-1187A-B-A-B, symbol TS-1187A-B-A-B:TS-1187A-B-A-B
- renumbered D9 to D3, J3 to J1, J4 to J2, J5 to J3, J6 to J4, R5 to R1, R16 to R5, TP3 to TP1, TP1 to TP3, U2 to U1
Connections:
- net +3.3V is gone; now on net +3V3: C1.1, C2.1, C3.1, C4.1, C5.1, C6.1, J1.2 (3.3V), J2.1 (Pin_1), J2.17 (Pin_17), R4.2, U1.1 (VLCD), U1.24 (VDD), U1.36 (VDD), U1.48 (VDD), U1.9 (VDDA)
- net GND: now also S2.A, S2.B
- net STM32_RESET: now also S2.C, S2.D
- no-connect marks 38 -> 36
